File: Electronics/WeMos Shield/D1MSHO.sch (EAGLE design)
At the start: 9 parts

Commit message: pcb design
Parts:
- C1: SPICEPREFIX (none) -> C
Changed lines of the file:
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@@
 <part name="U$2" library="freetronics-original" deviceset="5V" device=""/>
 <part name="GND2" library="freetronics-original" deviceset="GND" device=""/>
-<part name="C1" library="SparkFun-Capacitors" library_urn="urn:adsk.eagle:library:510" deviceset="1000UF" device="-RADIAL-5MM-25V-20%" package3d_urn="urn:adsk.eagle:package:37412/1" value="1mF"/>
+<part name="C1" library="SparkFun-Capacitors" library_urn="urn:adsk.eagle:library:510" deviceset="1000UF" device="-RADIAL-5MM-25V-20%" package3d_urn="urn:adsk.eagle:package:37412/1" value="1mF">
+<attribute name="SPICEPREFIX" value="C"/>
+</part>
 <part name="U$3" library="freetronics-original" deviceset="5V" device=""/>
 <part name="GND3" library="freetronics-original" deviceset="GND" device=""/>
